File: EKG_Design/ECG-PulseDetection.kicad_sch (KiCad schematic)
At the start: 8 parts, among them Q200 BC848C

Commit message: fixed the remaining DRC and ERC errors
Connections:
- net X: no longer names the net of D200.1 (A)
- no-connect marks 0 -> 1
Changed lines of the file:
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@@
 		(color 0 0 0 0)
+	)
+	(no_connect
+		(at 116.84 97.79)
 	)
 	(wire
@@
 		)
 	)
-	(label "X"
-		(at 116.84 97.79 0)
-		(effects
-			(font
-				(size 1.27 1.27)
-			)
-			(justify left bottom)
-		)
-	)
