File: EKG_Design/EKG_Design.kicad_sch (KiCad schematic)
At the start: 5 parts

Commit message: update ibom
Parts:
- H100, H101, H102, H103, PCB1: now fitted
Changed lines of the file:
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@@
 		(on_board yes)
 		(in_pos_files yes)
-		(dnp yes)
+		(dnp no)
 		(property "Reference" "H100"
 			(at 228.6 129.54 0)
@@
 		(on_board no)
 		(in_pos_files yes)
-		(dnp yes)
+		(dnp no)
 		(property "Reference" "PCB1"
 			(at 193.548 142.24 0)
@@
 		(on_board yes)
 		(in_pos_files yes)
-		(dnp yes)
+		(dnp no)
 		(property "Reference" "H101"
 			(at 254 129.54 0)
@@
 		(on_board yes)
 		(in_pos_files yes)
-		(dnp yes)
+		(dnp no)
 		(property "Reference" "H102"
 			(at 228.6 147.32 0)
@@
 		(on_board yes)
 		(in_pos_files yes)
-		(dnp yes)
+		(dnp no)
 		(property "Reference" "H103"
 			(at 254 147.32 0)
