File: AM Receiver/AM Receiver.kicad_sch (KiCad schematic)
At the start: 0 parts

Commit message: Updated AM Receiver Schematic with all Symbols. Footprint, manifest and data sheet still needed
Parts:
- added H1, H2, H3, H4: MountingHole_Pad, symbol Mechanical:MountingHole_Pad
- added PCB1: PCB, symbol AM_Receiver:PCB
Other:
- added sheet Am Schaltung (am-schaltung.kicad_sch)
- note added: "Info -->"
- note added: "Sheet 1 -->"

Commit message: Finished ECG Schematic and finished laying out the PCB
Parts:
- H1, H2, H3, H4: footprint (none) -> MountingHole:MountingHole_3.2mm_M3_Pad
Connections:
- net GND: now reaches H4.1
- net GND: now also H1.1, H2.1, H3.1
